Commit message: update

File: linorobot2_description/urdf/2wd_properties-orig.urdf.xacro (robot description, xacro)
@@ -12,5 +12,5 @@
   <xacro:property name="wheel_mass" value=".1" />
   <xacro:property name="wheel_torque" value="20" />
-  <xacro:property name="front_caster_wheel" value="false" />
+  <xacro:property name="front_caster_wheel" value="true" />
   <xacro:property name="rear_caster_wheel" value="true" />
   <xacro:property name="laser_pose">

File: linorobot2_description/urdf/robots/2wd-orig.urdf.xacro (robot description, xacro)
@@ -7,4 +7,6 @@
   <xacro:include filename="$(find linorobot2_description)/urdf/sensors/imu.urdf.xacro" />
   <xacro:include filename="$(find linorobot2_description)/urdf/sensors/generic_laser.urdf.xacro" />
+  <xacro:include filename="$(find linorobot2_description)/urdf/sensors/depth_sensor.urdf.xacro" />
+  <xacro:include filename="$(find linorobot2_description)/urdf/sensors/sonar.urdf.xacro" />
   <xacro:include filename="$(find linorobot2_description)/urdf/controllers/diff_drive.urdf.xacro" />
   <xacro:base
@@ -56,4 +58,11 @@
     <xacro:insert_block name="laser_pose" />
   </xacro:generic_laser>
+  <xacro:depth_sensor>
+    <xacro:insert_block name="depth_sensor_pose" />
+  </xacro:depth_sensor>
+  <xacro:sonar>
+    <xacro:insert_block name="sonar_pose"
+    />
+  </xacro:sonar>
   <xacro:diff_drive_controller
     wheel_separation="${wheel_pos_y * 2}"
