Commit message: work in progress

File: linorobot2_description/urdf/dome1.urdf.xacro (robot description, xacro)
@@ -169,5 +169,5 @@
     <parent link="base_link"/>
     <child link="laser"/>
-    <origin xyz="${laser_x_offset} 0 ${laser_z_offset}" rpy="0 0 0"/>
+    <origin xyz="${laser_x_offset} 0 ${laser_z_offset}" rpy="0 0 ${-pi/2}"/>
   </joint>
   <!-- IMU -->
@@ -197,5 +197,5 @@
       <origin xyz="0 0 0" rpy="0 0 0"/>
       <geometry>
-        <box size="0.010 0.010 0.010"/>
+        <box size="0.10 0.030 0.010"/>
       </geometry>
       <material name="red"/>

Commit message: trying to align everything

File: linorobot2_description/urdf/dome1.urdf.xacro (robot description, xacro)
@@ -49,8 +49,8 @@
   <!-- Base link (main robot body) -->
   <link name="base_link"/>
-  <joint name="base_footprint_to_base_link" type="fixed">
-    <parent link="base_footprint"/>
-    <child link="base_link"/>
-    <origin xyz="${base_link_x_offset} 0 ${bottom_plate_height}" rpy="0 0 0"/>
+  <joint name="base_link_to_base_footprint" type="fixed">
+    <parent link="base_link"/>
+    <child link="base_footprint"/>
+    <origin xyz="${-base_link_x_offset} 0 ${-bottom_plate_height}" rpy="0 0 0"/>
   </joint>
   <!-- Bottom plate -->
