Commit message: work in progress

File: linorobot2_description/urdf/2wd_properties.urdf.xacro (robot description, xacro)
@@ -12,8 +12,8 @@
   <xacro:property name="wheel_mass" value=".1" />
   <xacro:property name="wheel_torque" value="20" />
-  <xacro:property name="front_caster_wheel" value="true" />
+  <xacro:property name="front_caster_wheel" value="false" />
   <xacro:property name="rear_caster_wheel" value="true" />
   <xacro:property name="laser_pose">
-    <origin xyz="0.12 0 0.33" rpy="0 0 0"/>
+    <origin xyz="0.0 0 0.10" rpy="0 0 0"/>
   </xacro:property>
   <xacro:property name="depth_sensor_pose">

File: linorobot2_description/urdf/sensors/imu.urdf.xacro (robot description, xacro)
@@ -5,5 +5,5 @@
       <parent link="base_link"/>
       <child link="imu_link"/>
-      <origin xyz="0 0 .25" rpy="0 0 ${pi}"/>
+      <origin xyz="0 0 0" rpy="0 0 0"/>
     </joint>
     <gazebo reference="imu_link">

Commit message: Updating for new lidar

File: linorobot2_description/urdf/2wd_properties.urdf.xacro (robot description, xacro)
@@ -15,5 +15,5 @@
   <xacro:property name="rear_caster_wheel" value="true" />
   <xacro:property name="laser_pose">
-    <origin xyz="0.0 0 0.10" rpy="0 0 0"/>
+    <origin xyz="0.0 0 0.10" rpy="0 0 -${pi/2}"/>
   </xacro:property>
   <xacro:property name="depth_sensor_pose">

Commit message: synching up with hippo and getting rid of unneeded changes

File: linorobot2_description/urdf/2wd_properties.urdf.xacro (robot description, xacro)
@@ -12,14 +12,14 @@
   <xacro:property name="wheel_mass" value=".1" />
   <xacro:property name="wheel_torque" value="20" />
-  <xacro:property name="front_caster_wheel" value="false" />
+  <xacro:property name="front_caster_wheel" value="true" />
   <xacro:property name="rear_caster_wheel" value="true" />
   <xacro:property name="laser_pose">
-    <origin xyz="0.0 0 0.10" rpy="0 0 -${pi/2}"/>
+    <origin xyz="0.12 0 0.33" rpy="0 0 0"/>
   </xacro:property>
   <xacro:property name="depth_sensor_pose">
     <origin xyz="0.14 0.0 0.045" rpy="0 0 0"/>
   </xacro:property>
-  <xacro:property name="rear_camera_sensor_pose">
-    <origin xyz="-0.14 0.0 0.045" rpy="0 0 3.14159"/>
+  <xacro:property name="sonar_pose">
+    <origin xyz="0.15 0 0" rpy="0 0 0"/>
   </xacro:property>
 </robot>

File: linorobot2_description/urdf/robots/2wd.urdf.xacro (robot description, xacro)
@@ -8,5 +8,5 @@
   <xacro:include filename="$(find linorobot2_description)/urdf/sensors/generic_laser.urdf.xacro" />
   <xacro:include filename="$(find linorobot2_description)/urdf/sensors/depth_sensor.urdf.xacro" />
-  <xacro:include filename="$(find linorobot2_description)/urdf/sensors/camera.urdf.xacro" />
+  <xacro:include filename="$(find linorobot2_description)/urdf/sensors/sonar.urdf.xacro" />
   <xacro:include filename="$(find linorobot2_description)/urdf/controllers/diff_drive.urdf.xacro" />
   <xacro:base
@@ -61,10 +61,7 @@
     <xacro:insert_block name="depth_sensor_pose" />
   </xacro:depth_sensor>
-  <xacro:rgb_camera
-      parent="base_link"
-      name="rear_rgb_camera"
-      topic_name="rear_rgb_camera/image">
-    <xacro:insert_block name="rear_camera_sensor_pose" />
-  </xacro:rgb_camera>
+  <xacro:sonar>
+    <xacro:insert_block name="sonar_pose" />
+  </xacro:sonar>
   <xacro:diff_drive_controller
     wheel_separation="${wheel_pos_y * 2}"

File: linorobot2_description/urdf/robots/4wd.urdf.xacro (robot description, xacro)
@@ -7,5 +7,5 @@
   <xacro:include filename="$(find linorobot2_description)/urdf/sensors/generic_laser.urdf.xacro" />
   <xacro:include filename="$(find linorobot2_description)/urdf/sensors/depth_sensor.urdf.xacro" />
-  <xacro:include filename="$(find linorobot2_description)/urdf/sensors/camera.urdf.xacro" />
+  <xacro:include filename="$(find linorobot2_description)/urdf/sensors/sonar.urdf.xacro" />
   <xacro:include filename="$(find linorobot2_description)/urdf/controllers/skid_steer.urdf.xacro" />
   <xacro:base
@@ -60,10 +60,7 @@
     <xacro:insert_block name="depth_sensor_pose" />
   </xacro:depth_sensor>
-  <xacro:rgb_camera
-      parent="base_link"
-      name="rear_rgb_camera"
-      topic_name="rear_rgb_camera/image">
-    <xacro:insert_block name="rear_camera_sensor_pose" />
-  </xacro:rgb_camera>
+  <xacro:sonar>
+    <xacro:insert_block name="sonar_pose" />
+  </xacro:sonar>
   <xacro:diff_drive_controller
     wheel_separation="${wheel_pos_y * 2}"

File: linorobot2_description/urdf/robots/mecanum.urdf.xacro (robot description, xacro)
@@ -7,5 +7,5 @@
   <xacro:include filename="$(find linorobot2_description)/urdf/sensors/generic_laser.urdf.xacro" />
   <xacro:include filename="$(find linorobot2_description)/urdf/sensors/depth_sensor.urdf.xacro" />
-  <xacro:include filename="$(find linorobot2_description)/urdf/sensors/camera.urdf.xacro" />
+  <xacro:include filename="$(find linorobot2_description)/urdf/sensors/sonar.urdf.xacro" />
   <xacro:include filename="$(find linorobot2_description)/urdf/controllers/omni_drive.urdf.xacro" />
   <xacro:base
@@ -60,10 +60,7 @@
     <xacro:insert_block name="depth_sensor_pose" />
   </xacro:depth_sensor>
-  <xacro:rgb_camera
-      parent="base_link"
-      name="rear_rgb_camera"
-      topic_name="rear_rgb_camera/image">
-    <xacro:insert_block name="rear_camera_sensor_pose" />
-  </xacro:rgb_camera>
+  <xacro:sonar>
+    <xacro:insert_block name="sonar_pose" />
+  </xacro:sonar>
   <xacro:omni_drive_controller/>
 </robot>
